Commit message: added thumb pad

File: urdf/hdt_mk3_m.xacro (robot description, xacro)
@@ -596,4 +596,33 @@
 		</inertial>-->
 	</link>
+	<!-- thumb pad -->
+	<joint name="thumb_pad" type="fixed">
+		<origin xyz="0 0 0" rpy="0 0 0"/>
+		<parent link="thumb_base"/>
+		<child link="thumb_pad"/>
+	</joint>
+	<link name="thumb_pad">
+		<!--<collision>
+			<origin xyz="0 0 0" rpy="0 0 0"/>
+			<geometry>
+				<mesh filename="package://hdt_mk3_m_description/meshes/hdt_mk3_m_thumb_pad.STL"/>
+			</geometry>
+		</collision>-->
+		<visual>
+			<origin xyz="0 0 0.0" rpy="0 0 0"/>
+			<geometry>
+				<mesh filename="package://hdt_mk3_m_description/meshes/hdt_mk3_m_thumb_pad.STL"/>
+			</geometry>
+			<material name="yellow"/>
+		</visual>
+		<!--<inertial>
+			<origin xyz="0 -0.08326 -0.00539" rpy="0 0 0"/>
+			<mass value="0.56756"/>
+			<inertia
+			ixx="0.001727803" ixy="0.000001205" ixz="0.0"
+			iyy="0.000549457" iyz="-0.000101997"
+			izz="0.001418031"/>
+		</inertial>-->
+	</link>
 	<!-- thumb prox -->
 	<joint name="thumb_prox" type="revolute">
